Commit message: done with resizing

File: catkin_ws/src/fusion/robot_description/urdf/fusion.urdf (robot description, URDF)
Before this commit: robot fusion, 27 links, 26 joints
Links:
- link chassis: geometry collision box size=1.74 0.896 0.05; collision box size=1.74 1.0 0.05
- link front_left_wheel: geometry collision sphere radius=0.48; visual mesh filename=package://fusion/robot_description/meshes/fusion/wheel.dae scale=0.013 0.013 0.013
- link front_right_wheel: geometry collision sphere radius=0.48; visual mesh filename=package://fusion/robot_description/meshes/fusion/wheel.dae scale=0.013 0.013 0.013
- link rear_left_wheel: geometry collision sphere radius=0.48; visual mesh filename=package://fusion/robot_description/meshes/fusion/wheel.dae scale=0.013 0.013 0.013
- link rear_right_wheel: geometry collision sphere radius=0.48; visual mesh filename=package://fusion/robot_description/meshes/fusion/wheel.dae scale=0.013 0.013 0.013
- link steering_wheel: geometry visual mesh filename=package://fusion/robot_description/meshes/fusion/steering_w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 scale=0.013 0.013 0.013
Joints:
- joint back_camera_joint: origin xyz=0 1.75 2.42 rpy=0 0.05 1.5707 -> xyz=0 1.65 1.82 rpy=0 0.05 1.5707
- joint camera_optical_joint: origin xyz=0 -0.7 2.42 rpy=0 0 -1.57 -> xyz=0 -0.5 1.81 rpy=0 0 -1.57
- joint center_laser_joint: origin xyz=0 0.1 3.00 rpy=0 0.05 -1.5707 -> xyz=0 0.1 1.95 rpy=0 0.05 -1.5707
- joint front_camera_joint: origin xyz=0 -0.7 2.42 rpy=0 0.05 -1.5707 -> xyz=0 -0.6 1.83 rpy=0 0.05 -1.5707
- joint front_left_laser_joint: origin xyz=1.5 -2 1.3 rpy=0 0.22 0 -> xyz=1.2 -1.8 1.0 rpy=0 0.22 0
- joint front_left_steer_joint: origin xyz=1.3806 -2.538 0.54 rpy=0 0 0 -> xyz=1.1 -2.0 0.54 rpy=0 0 0
- joint front_right_laser_joint: origin xyz=-1.5 -2 1.3 rpy=0 0.22 3.14 -> xyz=-1.2 -1.8 1.0 rpy=0 0.22 3.14
- joint front_right_steer_joint: origin xyz=-1.3806 -2.538 0.54 rpy=0 0 0 -> xyz=-1.1 -2.0 0.54 rpy=0 0 0
- joint left_camera_joint: origin xyz=0.8 -0.7 2.42 rpy=0 0.05 -1.94 -> xyz=0.8 -0.6 1.83 rpy=0 0.05 -1.5707
- joint rear_left_wheel_joint: origin xyz=1.2474 2.36 0.54 rpy=0 0 0 -> xyz=1.1 1.8 0.54 rpy=0 0 0
- joint rear_right_wheel_joint: origin xyz=-1.2474 2.36 0.54 rpy=0 0 0 -> xyz=-1.1 1.8 0.54 rpy=0 0 0
- joint right_camera_joint: origin xyz=-0.8 -0.7 2.42 rpy=0 0.05 -1.20 -> xyz=-0.8 -0.6 1.83 rpy=0 0.05 -1.5707
- joint steering_joint: origin xyz=0.6439212 -1.1301624 1.7788374 rpy=-1.302101 0 0 -> xyz=0.6439212 -0.8 1.3 rpy=-1.302101 0 0
- joint velodyne_joint: origin xyz=0 -0.7 2.42 rpy=0 0 -1.57 -> xyz=0 -0.5 1.86 rpy=0 0 -1.57

Commit message: add imu and gps sensors

File: catkin_ws/src/fusion/robot_description/urdf/fusion.urdf (robot description, URDF)
Before this commit: robot fusion, 27 links, 26 joints
Links:
- removed link back_left_far_sonar_link
- removed link back_left_middle_sonar_link
- removed link back_right_far_sonar_link
- removed link back_right_middle_sonar_link
- removed link camera_link
- removed link center_laser_link
- removed link front_left_far_sonar_link
- removed link front_left_laser_link
- removed link front_left_middle_sonar_link
- removed link front_right_far_sonar_link
- removed link front_right_laser_link
- removed link front_right_middle_sonar_link
- added link base_footprint, mass 0.0001; visual box size=0.001 0.001 0.001
- added link base_topprint; visual box size=0.001 0.001 0.001
- added link gps_link, mass 1; collision box size=0.1 0.1 0.1; visual box size=0.1 0.1 0.1
Joints:
- removed joint back_left_far_sonar_joint
- removed joint back_left_middle_sonar_joint
- removed joint back_right_far_sonar_joint
- removed joint back_right_middle_sonar_joint
- removed joint camera_optical_joint
- removed joint center_laser_joint
- removed joint front_left_far_sonar_joint
- removed joint front_left_laser_joint
- removed joint front_left_middle_sonar_joint
- removed joint front_right_far_sonar_joint
- removed joint front_right_laser_joint
- removed joint front_right_middle_sonar_joint
- added joint base_footprint_joint: type fixed, parent base_footprint, child base_link, origin xyz=0 0 0 rpy=0 0 0
- added joint base_topprint_joint: type fixed, parent base_topprint, child base_footprint, origin xyz=0 0 -2 rpy=0 0 0
- added joint gps_joint: type fixed, parent chassis, child gps_link, origin xyz=0.05 0 0.15 rpy=0 0 0, axis 0 0 0

Commit message: add gravity off to camera link

File: catkin_ws/src/fusion/robot_description/urdf/fusion.urdf (robot description, URDF)
Before this commit: robot fusion, 18 links, 17 joints
Links:
- added link camera_link, mass 1
Joints:
- added joint camera_optical_joint: type fixed, parent chassis, child camera_link, origin xyz=0 -0.5 1.81 rpy=0 0 -1.57, axis 0 1 0

Commit message: convert data_collection to class

File: catkin_ws/src/fusion/robot_description/urdf/fusion.urdf (robot description, URDF)
Before this commit: robot fusion, 19 links, 18 joints
Links:
- removed link base_footprint
- removed link base_topprint
- removed link camera_link
- link front_left_wheel: geometry collision sphere radius=0.47; visual mesh filename=package://fusion/robot_description/meshes/fusion/wheel.dae scale=0.014 0.014 0.014
- link front_right_wheel: geometry collision sphere radius=0.47; visual mesh filename=package://fusion/robot_description/meshes/fusion/wheel.dae scale=0.014 0.014 0.014
- link rear_left_wheel: geometry collision sphere radius=0.47; visual mesh filename=package://fusion/robot_description/meshes/fusion/wheel.dae scale=0.014 0.014 0.014
- link rear_right_wheel: geometry collision sphere radius=0.47; visual mesh filename=package://fusion/robot_description/meshes/fusion/wheel.dae scale=0.014 0.014 0.014
Joints:
- removed joint base_footprint_joint
- removed joint base_topprint_joint
- removed joint camera_optical_joint
- joint base_link_connection: origin xyz=0 0 0 rpy=0 0 1.57 -> xyz=0 0 0 rpy=0 0 0
- joint steering_joint: origin xyz=0.6439212 -0.8 1.3 rpy=-1.302101 0 0 -> xyz=0.5439212 -0.8 1.3 rpy=-1.302101 0 0

Commit message: edit road.png and fusion.urdf

File: catkin_ws/src/fusion/robot_description/urdf/fusion.urdf (robot description, URDF)
Before this commit: robot fusion, 16 links, 15 joints
Links:
- removed link velodyne_link
- link front_left_wheel: geometry collision cylinder length=0.47 radius=0.47; visual mesh filename=package://fusion/robot_description/meshes/fusion/wheel.dae scale=0.014 0.014 0.014
- link front_right_wheel: geometry collision cylinder length=0.47 radius=0.47; visual mesh filename=package://fusion/robot_description/meshes/fusion/wheel.dae scale=0.014 0.014 0.014
- link rear_left_wheel: geometry collision cylinder length=0.47 radius=0.47; visual mesh filename=package://fusion/robot_description/meshes/fusion/wheel.dae scale=0.014 0.014 0.014
- link rear_right_wheel: geometry collision cylinder length=0.47 radius=0.47; visual mesh filename=package://fusion/robot_description/meshes/fusion/wheel.dae scale=0.014 0.014 0.014
Joints:
- removed joint velodyne_joint
- joint base_link_connection: origin xyz=0 0 0 rpy=0 0 0 -> xyz=0 0 0 rpy=0 0 1.57079632
- joint imu_joint: parent chassis -> base_link

Commit message: add ground_plane png & edit test_saliency

File: catkin_ws/src/fusion/robot_description/urdf/fusion.urdf (robot description, URDF)
Before this commit: robot fusion, 15 links, 14 joints
Links:
- link front_left_wheel: geometry collision sphere radius=0.47; visual mesh filename=package://fusion/robot_description/meshes/fusion/wheel.dae scale=0.014 0.014 0.014
- link front_right_wheel: geometry collision sphere radius=0.47; visual mesh filename=package://fusion/robot_description/meshes/fusion/wheel.dae scale=0.014 0.014 0.014
- link gps_link: geometry 
- link rear_left_wheel: geometry collision sphere radius=0.47; visual mesh filename=package://fusion/robot_description/meshes/fusion/wheel.dae scale=0.014 0.014 0.014
- link rear_right_wheel: geometry collision sphere radius=0.47; visual mesh filename=package://fusion/robot_description/meshes/fusion/wheel.dae scale=0.014 0.014 0.014
Joints:
- joint base_link_connection: origin xyz=0 0 0 rpy=0 0 1.57079632 -> xyz=0 0 -0.3 rpy=0 0 1.57079632
